File: trap-pcb.sch (KiCad schematic (older format))
At the start: 80 parts, among them J1 Conn_01x15, J2 Conn_01x15, M1 Motor_DC, Q1 Q_NMOS_GSD, Q2 Q_NMOS_GSD, Q3 Q_NMOS_GSD, Q4 Q_NMOS_GSD, Q5 Q_NMOS_GSD, Q6 Q_NMOS_GSD, Q7 Q_NMOS_GSD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

Commit message: Updated JLC and DigiKey parts
Parts:
- 6V_1, VCC_1: DigiKey (none) -> 455-1704-ND; DigiKey  455-1704-ND -> (none)
- J1, J2: DigiKey (none) -> S7013-ND
- M1: footprint Connector_JST:JST_XH_B2B-XH-A_1x02_P2.50mm_Vertical -> Connector_JST:JST_PH_B2B-PH-K_1x02_P2.00mm_Vertical; DigiKey (none) -> 455-1705-ND
- PIR_1, PIR_2, PIR_3, Servo_1, Servo_2, Servo_3: Manufacturer B3B-PH-K-S(LF)(SN) -> (none); Manufacturer Part # (none) -> B3B-PH-K-S(LF)(SN)
- SW1: DigiKey (none) -> 401-1985-ND; Manufacturer Part # (none) -> D6C40 F2 LFS
- SW2: DigiKey (none) -> 455-1704-ND; Manufacturer Part # (none) -> EG1903-ND
- Ultrasonic_Cage1: Manufacturer Part B5B-PH-K-S(LF)(SN) -> (none); Manufacturer Part # (none) -> B5B-PH-K-S(LF)(SN)
- Ultrasonic_Trap1: Manufacturer Part # (none) -> B5B-PH-K-S(LF)(SN); Maufacturer B5B-PH-K-S(LF)(SN) -> (none)
- VDD1: renamed from 3.3V_1; DigiKey (none) -> 455-1704-ND; DigiKey  455-1704-ND -> (none)
Connections:
- net +3V3 renamed VDD
Changed lines of the file:
@@
 F 3 "~" H 10350 5150 50  0001 C CNN
 F 4 "455-1705-ND" H 10350 5150 50  0001 C CNN "DigiKey"
-F 5 "B3B-PH-K-S(LF)(SN)" H 10350 5150 50  0001 C CNN "Manufacturer"
+F 5 "" H 10350 5150 50  0001 C CNN "Manufacturer"
+F 6 "B3B-PH-K-S(LF)(SN)" H 10350 5150 50  0001 C CNN "Manufacturer Part #"
 	1    10350 5150
 	1    0    0    -1
@@
 F 2 "Connector_PinHeader_2.54mm:PinHeader_1x15_P2.54mm_Vertical" H 800 2500 50  0001 C CNN
 F 3 "~" H 800 2500 50  0001 C CNN
+F 4 "S7013-ND" H 800 2500 50  0001 C CNN "DigiKey"
 	1    800  2500
 	-1   0    0    -1
@@
 F 2 "Connector_PinHeader_2.54mm:PinHeader_1x15_P2.54mm_Vertical" H 4700 3000 50  0001 C CNN
 F 3 "~" H 4700 3000 50  0001 C CNN
+F 4 "S7013-ND" H 4700 3000 50  0001 C CNN "DigiKey"
 	1    4700 3000
 	1    0    0    -1
@@
 F 0 "M1" H 6308 6146 50  0000 L CNN
 F 1 "Motor_DC" H 6308 6055 50  0000 L CNN
-F 2 "Connector_JST:JST_XH_B2B-XH-A_1x02_P2.50mm_Vertical" H 6150 6060 50  0001 C CNN
+F 2 "Connector_JST:JST_PH_B2B-PH-K_1x02_P2.00mm_Vertical" H 6150 6060 50  0001 C CNN
 F 3 "~" H 6150 6060 50  0001 C CNN
+F 4 "455-1705-ND" H 6150 6150 50  0001 C CNN "DigiKey"
 	1    6150 6150
 	1    0    0    -1
@@
 SCL
 $Comp
-L trap-pcb-rescue:+3.3V-power #PWR0139
+L power:VDD #PWR0139
 U 1 1 60365B2B
 P 6950 750
 F 0 "#PWR0139" H 6950 600 50  0001 C CNN
-F 1 "+3.3V" H 6965 923 50  0000 C CNN
+F 1 "VDD" H 6965 923 50  0000 C CNN
 F 2 "" H 6950 750 50  0001 C CNN
 F 3 "" H 6950 750 50  0001 C CNN
@@
 F 2 "Button_Switch_THT:Push_E-Switch_KS01Q01" H 1250 4750 50  0001 C CNN
 F 3 "~" H 1250 4750 50  0001 C CNN
+F 4 "401-1985-ND" H 1250 4750 50  0001 C CNN "DigiKey"
+F 5 "D6C40 F2 LFS" H 1250 4750 50  0001 C CNN "Manufacturer Part #"
 	1    1250 4750
 	0    -1   -1   0
@@
 F 3 "~" H 10500 2500 50  0001 C CNN
 F 4 "455-1707-ND" H 10500 2500 50  0001 C CNN "DigiKey"
-F 5 "B5B-PH-K-S(LF)(SN)" H 10500 2500 50  0001 C CNN "Maufacturer"
+F 5 "" H 10500 2500 50  0001 C CNN "Maufacturer"
 F 6 "" H 10500 2500 50  0001 C CNN "JLCPCB"
+F 7 "B5B-PH-K-S(LF)(SN)" H 10500 2500 50  0001 C CNN "Manufacturer Part #"
 	1    10500 2500
 	1    0    0    -1
@@
 F 3 "~" H 9700 1350 50  0001 C CNN
 F 4 "455-1707-ND" H 9700 1350 50  0001 C CNN "DigiKey"
-F 5 "B5B-PH-K-S(LF)(SN)" H 9700 1350 50  0001 C CNN "Manufacturer Part"
+F 5 "" H 9700 1350 50  0001 C CNN "Manufacturer Part"
 F 6 "" H 9700 1350 50  0001 C CNN "JLCPCB"
+F 7 "B5B-PH-K-S(LF)(SN)" H 9700 1350 50  0001 C CNN "Manufacturer Part #"
 	1    9700 1350
 	1    0    0    -1
@@
 F 2 "trap-pcb:EG1218" H 4650 5165 60  0001 C CNN
 F 3 "" H 4350 5150 60  0000 C CNN
+F 4 "455-1704-ND" H 4350 5150 50  0001 C CNN "DigiKey"
+F 5 "EG1903-ND" H 4350 5150 50  0001 C CNN "Manufacturer Part #"
 	1    4350 5150
 	1    0    0    -1
@@
 F 3 "~" H 5050 1400 50  0001 C CNN
 F 4 "B2B-PH-K-S(LF)(SN)" H 5050 1400 50  0001 C CNN "Manufacturer Part #"
-F 5 "455-1704-ND" H 5050 1400 50  0001 C CNN "DigiKey "
+F 5 "" H 5050 1400 50  0001 C CNN "DigiKey "
 F 6 "" H 5050 1400 50  0001 C CNN "JLCPCB"
+F 7 "455-1704-ND" H 5050 1400 50  0001 C CNN "DigiKey"
 	1    5050 1400
 	-1   0    0    1
@@
 $EndComp
 $Comp
-L Connectors:Conn_01x02 3.3V_1
+L Connectors:Conn_01x02 VDD1
 U 1 1 5FA929AC
 P 6500 1400
-F 0 "3.3V_1" H 6600 1100 50  0000 C CNN
+F 0 "VDD1" H 6600 1100 50  0000 C CNN
 F 1 "CONN HEADER VERT 2POS 2MM" H 6600 1200 50  0001 C CNN
 F 2 "Connector_JST:JST_PH_B2B-PH-K_1x02_P2.00mm_Vertical" H 6500 1400 50  0001 C CNN
 F 3 "~" H 6500 1400 50  0001 C CNN
 F 4 "B2B-PH-K-S(LF)(SN)" H 6500 1400 50  0001 C CNN "Manufacturer Part #"
-F 5 "455-1704-ND" H 6500 1400 50  0001 C CNN "DigiKey "
+F 5 "" H 6500 1400 50  0001 C CNN "DigiKey "
 F 6 "" H 6500 1400 50  0001 C CNN "JLCPCB"
+F 7 "455-1704-ND" H 6500 1400 50  0001 C CNN "DigiKey"
 	1    6500 1400
 	-1   0    0    1
@@
 F 3 "~" H 7900 1400 50  0001 C CNN
 F 4 "B2B-PH-K-S(LF)(SN)" H 7900 1400 50  0001 C CNN "Manufacturer Part #"
-F 5 "455-1704-ND" H 7900 1400 50  0001 C CNN "DigiKey "
+F 5 "" H 7900 1400 50  0001 C CNN "DigiKey "
 F 6 "" H 7900 1400 50  0001 C CNN "JLCPCB"
+F 7 "455-1704-ND" H 7900 1400 50  0001 C CNN "DigiKey"
 	1    7900 1400
 	-1   0    0    1
@@
 F 3 "~" H 10350 5500 50  0001 C CNN
 F 4 "455-1705-ND" H 10350 5500 50  0001 C CNN "DigiKey"
-F 5 "B3B-PH-K-S(LF)(SN)" H 10350 5500 50  0001 C CNN "Manufacturer"
+F 5 "" H 10350 5500 50  0001 C CNN "Manufacturer"
+F 6 "B3B-PH-K-S(LF)(SN)" H 10350 5500 50  0001 C CNN "Manufacturer Part #"
 	1    10350 5500
 	1    0    0    -1
@@
 F 3 "~" H 10350 5850 50  0001 C CNN
 F 4 "455-1705-ND" H 10350 5850 50  0001 C CNN "DigiKey"
-F 5 "B3B-PH-K-S(LF)(SN)" H 10350 5850 50  0001 C CNN "Manufacturer"
+F 5 "" H 10350 5850 50  0001 C CNN "Manufacturer"
+F 6 "B3B-PH-K-S(LF)(SN)" H 10350 5850 50  0001 C CNN "Manufacturer Part #"
 	1    10350 5850
 	1    0    0    -1
@@
 F 3 "~" H 1000 6550 50  0001 C CNN
 F 4 "455-1705-ND" H 1000 6550 50  0001 C CNN "DigiKey"
-F 5 "B3B-PH-K-S(LF)(SN)" H 1000 6550 50  0001 C CNN "Manufacturer"
+F 5 "" H 1000 6550 50  0001 C CNN "Manufacturer"
+F 6 "B3B-PH-K-S(LF)(SN)" H 1000 6550 50  0001 C CNN "Manufacturer Part #"
 	1    1000 6550
 	-1   0    0    1
@@
 F 3 "~" H 1000 7200 50  0001 C CNN
 F 4 "455-1705-ND" H 1000 7200 50  0001 C CNN "DigiKey"
-F 5 "B3B-PH-K-S(LF)(SN)" H 1000 7200 50  0001 C CNN "Manufacturer"
+F 5 "" H 1000 7200 50  0001 C CNN "Manufacturer"
+F 6 "B3B-PH-K-S(LF)(SN)" H 1000 7200 50  0001 C CNN "Manufacturer Part #"
 	1    1000 7200
 	-1   0    0    1
@@
 F 3 "~" H 2300 7200 50  0001 C CNN
 F 4 "455-1705-ND" H 2300 7200 50  0001 C CNN "DigiKey"
-F 5 "B3B-PH-K-S(LF)(SN)" H 2300 7200 50  0001 C CNN "Manufacturer"
+F 5 "" H 2300 7200 50  0001 C CNN "Manufacturer"
+F 6 "B3B-PH-K-S(LF)(SN)" H 2300 7200 50  0001 C CNN "Manufacturer Part #"
 	1    2300 7200
 	-1   0    0    1
